File: ESP32_robot.kicad_pcb (KiCad board)
At the start: 2 copper layers, 60.3 x 38.2 mm, 30 parts, among them J1 USB_C_Receptacle_USB2.0, J2 Conn_01x08_Male, J3 01x02, J4 Conn_01x08_Male, J5 01x02, SW1 SW_Push, SW2 SW_Push, U1 ESP32-S2-MINI-1-N4, U2 LM1117-3.3

Commit message: hopefully the latest
Connections:
- U1 pad 20: USB_N -> unconnected-(U1-Pad20)
- U1 pad 21: USB_P -> unconnected-(U1-Pad21)
- U1 pad 23: unconnected-(U1-Pad23) -> USB_N
- U1 pad 24: unconnected-(U1-Pad24) -> USB_P
Routing:
- net USB_P: track 8.94 -> 10.3 mm
- net USB_N: track 9.02 -> 10.2 mm
Changed lines of the file:
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@@
       (outputformat 1)
       (mirror false)
-      (drillshape 1)
+      (drillshape 0)
       (scaleselection 1)
-      (outputdirectory "")
+      (outputdirectory "juni2022")
     )
   )
@@
   (net 39 "/Header_9")
   (net 40 "/Header_10")
-  (net 41 "unconnected-(U1-Pad23)")
-  (net 42 "unconnected-(U1-Pad24)")
+  (net 41 "unconnected-(U1-Pad20)")
+  (net 42 "unconnected-(U1-Pad21)")
   (net 43 "Net-(D1-Pad2)")
   (net 44 "Net-(D1-Pad3)")
@@
       (net 40 "/Header_10") (pinfunction "IO15") (pintype "bidirectional"))
     (pad "20" smd rect (at -2.55 9.288513) (size 0.4064 0.8128) (layers "F.Cu" "F.Paste" "F.Mask")
-      (net 18 "USB_N") (pinfunction "IO16") (pintype "bidirectional"))
+      (net 41 "unconnected-(U1-Pad20)") (pinfunction "IO16") (pintype "bidirectional+no_connect"))
     (pad "21" smd rect (at -1.699999 9.288513) (size 0.4064 0.8128) (layers "F.Cu" "F.Paste" "F.Mask")
-      (net 19 "USB_P") (pinfunction "IO17") (pintype "bidirectional"))
+      (net 42 "unconnected-(U1-Pad21)") (pinfunction "IO17") (pintype "bidirectional+no_connect"))
     (pad "22" smd rect (at -0.850001 9.288513) (size 0.4064 0.8128) (layers "F.Cu" "F.Paste" "F.Mask")
       (net 45 "unconnected-(U1-Pad22)") (pinfunction "IO18") (pintype "bidirectional+no_connect"))
     (pad "23" smd rect (at 0 9.288513) (size 0.4064 0.8128) (layers "F.Cu" "F.Paste" "F.Mask")
-      (net 41 "unconnected-(U1-Pad23)") (pinfunction "IO19") (pintype "bidirectional+no_connect"))
+      (net 18 "USB_N") (pinfunction "IO19") (pintype "bidirectional"))
     (pad "24" smd rect (at 0.850001 9.288513) (size 0.4064 0.8128) (layers "F.Cu" "F.Paste" "F.Mask")
-      (net 42 "unconnected-(U1-Pad24)") (pinfunction "IO20") (pintype "bidirectional+no_connect"))
+      (net 19 "USB_P") (pinfunction "IO20") (pintype "bidirectional"))
     (pad "25" smd rect (at 1.699999 9.288513) (size 0.4064 0.8128) (layers "F.Cu" "F.Paste" "F.Mask")
       (net 10 "/Header_1") (pinfunction "IO21") (pintype "bidirectional"))
@@
   (segment (start 113.679999 56.488515) (end 121.918515 56.488515) (width 0.25) (layer "F.Cu") (net 17))
   (segment (start 121.918515 56.488515) (end 130.43 65) (width 0.25) (layer "F.Cu") (net 17))
-  (segment (start 103.5812 68.881) (end 103.5812 63.3888) (width 0.2) (layer "F.Cu") (net 18))
-  (segment (start 104.13 62.84) (end 104.13 60.088513) (width 0.2) (layer "F.Cu") (net 18))
-  (segment (start 103.5812 63.3888) (end 104.13 62.84) (width 0.2) (layer "F.Cu") (net 18))
-  (segment (start 104.980001 63.380001) (end 105.2576 63.6576) (width 0.2) (layer "F.Cu") (net 19))
-  (segment (start 105.2576 63.6576) (end 105.2576 68.9102) (width 0.2) (layer "F.Cu") (net 19))
-  (segment (start 104.980001 60.088513) (end 104.980001 63.380001) (width 0.2) (layer "F.Cu") (net 19))
+  (segment (start 106.880001 63.883256) (end 104.179799 66.583458) (width 0.2) (layer "F.Cu") (net 18))
+  (segment (start 104.179799 68.282401) (end 103.5812 68.881) (width 0.2) (layer "F.Cu") (net 18))
+  (segment (start 106.68 60.698114) (end 106.880001 60.898115) (width 0.2) (layer "F.Cu") (net 18))
+  (segment (start 106.880001 60.898115) (end 106.880001 63.883256) (width 0.2) (layer "F.Cu") (net 18))
+  (segment (start 104.179799 66.583458) (end 104.179799 68.282401) (width 0.2) (layer "F.Cu") (net 18))
+  (segment (start 106.68 60.088513) (end 106.68 60.698114) (width 0.2) (layer "F.Cu") (net 18))
+  (segment (start 107.530001 60.088513) (end 107.530001 60.698114) (width 0.2) (layer "F.Cu") (net 19))
+  (segment (start 107.33 60.898115) (end 107.33 64.069657) (width 0.2) (layer "F.Cu") (net 19))
+  (segment (start 104.629801 68.282401) (end 105.2576 68.9102) (width 0.2) (layer "F.Cu") (net 19))
+  (segment (start 104.629801 66.769856) (end 104.629801 68.282401) (width 0.2) (layer "F.Cu") (net 19))
+  (segment (start 107.530001 60.698114) (end 107.33 60.898115) (width 0.2) (layer "F.Cu") (net 19))
+  (segment (start 107.33 64.069657) (end 104.629801 66.769856) (width 0.2) (layer "F.Cu") (net 19))
   (segment (start 99.680001 50.538515) (end 99.361485 50.538515) (width 0.25) (layer "F.Cu") (net 22))
   (segment (start 83.85 57.1) (end 82.8 56.05) (width 0.25) (layer "F.Cu") (net 22))
